File: Buck Regulator_secondary.brd (EAGLE design)
At the start: 42.5 x 35 mm, 26 parts, among them IC1 LM5017

Commit message: update
Parts:
- R4: value 2k -> 20k
- moved C7 12.3 mm to (15.9, 25.0), turned to 180 degrees
- moved C4 12.0 mm to (19.5, 23.9), turned to 0 degrees
- moved R2 9.33 mm to (15.9, 27.4), turned to 180 degrees
- moved TP2 9.21 mm to (23.3, 24.1)
- moved R3 9.04 mm to (19.3, 27.4), turned to 180 degrees
- moved R4 8.85 mm to (15.9, 22.8), turned to 180 degrees
- moved TP5 7.63 mm to (14.8, 16.8)
- moved C2 7.28 mm to (18.3, 20.4), flipped to the top, turned to 180 degrees
- moved C5 7.12 mm to (12.9, 18.0), flipped to the top
- moved C3 7.00 mm to (18.1, 17.8), flipped to the top
- moved TP3 6.91 mm to (30.0, 20.9)
- moved R1 6.65 mm to (29.5, 23.3)
- moved IC1 6.11 mm to (24.0, 19.3)
- moved R5 4.68 mm to (29.5, 22.2), turned to 0 degrees
- moved R6 4.61 mm to (29.5, 19.7), turned to 180 degrees
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Connections:
- net +12V: now also X2.1; no longer X2.2
- net GND: now also X2.2; no longer X2.1
Routing:
- net GND: track 51.5 -> 5.12 mm, vias 1 -> 3
- net VIN_HV: track 25.5 -> 5.93 mm
- net +12V: track 33.1 -> 14.7 mm, vias 1 -> 0
- net N$29: track 25.7 -> 11.0 mm, vias 1 -> 0
- net FB: track 20.0 -> 12.7 mm
- net N$1: track 7.55 -> 4.03 mm
- net N$23: track 4.87 -> 2.14 mm, vias 1 -> 0
- net N$31: track 1.80 -> 3.79 mm
- net N$2: track 7.17 -> 5.70 mm
- net N$28: track 5.22 -> 4.82 mm, vias 1 -> 0
- added copper zone on layer 1, net +12V
- added copper zone on layer 1, net GND
- added copper zone on layer 16, net GND
- added copper zone on layer 1, net N$29
- added copper zone on layer 1, net VIN_HV
Other:
- board size 42.5 x 35 mm -> 43 x 35 mm
