File: Buck Regulator_secondary.sch (EAGLE design)
At the start: 26 parts, among them IC1 LM5017

Commit message: update
Parts:
- R4: value 2k -> 20k
Connections:
- net +12V: now also X2-1.KL; no longer X2-2.KL
- net GND: now also X2-2.KL; no longer X2-1.KL
Other:
- moved on the sheet: X2-1, X2-2
